Commit message: Merge engineer updates (Fixed Sim and MoveIt)

File: brain_pc/src/mycobot_320pi_description/urdf/mycobot_320pi.urdf.xacro (robot description, xacro)
@@ -38,5 +38,5 @@
     </transmission>
     <!-- Links -->
-    <link name="base_link"/>
+    <link name="world"/>
     <!-- Base Link-->
     <link name="base_plate">
@@ -297,5 +297,5 @@
     <!-- virtual Joints -->
     <joint name="virtual_joint" type="fixed">
-        <parent link="base_link"/>
+        <parent link="world"/>
         <child link="base_plate"/>
         <origin xyz="0 0 0" rpy="0 0 0"/>

Commit message: merge

File: brain_pc/src/mycobot_320pi_description/urdf/mycobot_320pi.urdf.xacro (robot description, xacro)
@@ -1,4 +1,6 @@
 <?xml version="1.0"?>
 <robot xmlns:xacro="http://www.ros.org/wiki/xacro" name="mycobot_320pi">
+    <!-- Start GZ or Ignition depending on ROS 2 Version -->
+    <xacro:arg name="is_ignition" default="true"/>
     <!-- Load Simulated or Real Hardware Interfaces -->
     <xacro:arg name="is_sim" default="true"/>
@@ -21,20 +23,4 @@
         </inertial>
     </xacro:macro>
-    <xacro:macro name="default_transmission" params="number">
-        <transmission name="transmission_${number}">
-            <plugin>transmission_interface/SimpleTransmission</plugin>
-            <actuator name="motor_${number}" role="actuator1"/>
-            <joint name="joint_${number}"    role="joint1">
-                <mechanical_reduction>1.0</mechanical_reduction>
-            </joint>
-        </transmission>
-    </xacro:macro>
-    <transmission name="transmission_gripper_master">
-        <plugin>transmission_interface/SimpleTransmission</plugin>
-        <actuator name="motor_gripper_master" role="actuator1"/>
-        <joint name="left_jaw_joint_1" role="joint1">
-            <mechanical_reduction>1.0</mechanical_reduction>
-        </joint>
-    </transmission>
     <!-- Links -->
     <link name="world"/>
@@ -420,10 +406,3 @@
         <mimic joint="left_jaw_joint_1" multiplier="1.0" offset="0" />
     </joint>
-    <!-- Transmissions-->
-    <xacro:default_transmission number="1"/>
-    <xacro:default_transmission number="2"/>
-    <xacro:default_transmission number="3"/>
-    <xacro:default_transmission number="4"/>
-    <xacro:default_transmission number="5"/>
-    <xacro:default_transmission number="6"/>
 </robot>

File: brain_pc/src/mycobot_320pi_description/urdf/mycobot_320pi_gazebo.xacro (robot description, xacro)
@@ -1,11 +1,18 @@
 <?xml version="1.0"?>
-<robot xmlns:xacro="http://www.ros.org/wiki/xacro" name="robot_2030a">
-    <!-- Gazebo ros2_control plugin -->
-    <gazebo>
-      <plugin filename="libgazebo_ros2_control.so" name="gazebo_ros2_control">
-        <robot_param>robot_description</robot_param>
-        <robot_param_node>robot_state_publisher</robot_param_node>
+<robot xmlns:xacro="http://www.ros.org/wiki/xacro" name="mycobot_320pi">
+  <!-- ROS 2 Control -->
+  <gazebo>
+    <!-- ROS 2 Humble -->
+    <xacro:if value="$(arg is_ignition)">
+      <plugin filename="ign_ros2_control-system" name="ign_ros2_control::IgnitionROS2ControlPlugin">
         <parameters>$(find mycobot_320pi_controller)/config/mycobot_320pi_controllers.yaml</parameters>
       </plugin>
-    </gazebo>
+    </xacro:if>
+    <!-- ROS 2 Iron or above -->
+    <xacro:unless value="$(arg is_ignition)">
+      <plugin filename="gz_ros2_control-system" name="gz_ros2_control::GazeboSimROS2ControlPlugin">
+        <parameters>$(find mycobot_320pi_controller)/config/mycobot_320pi_controllers.yaml</parameters>
+      </plugin>
+    </xacro:unless>
+</gazebo>
 </robot>

File: brain_pc/src/mycobot_320pi_description/urdf/mycobot_320pi_ros2_control.xacro (robot description, xacro)
@@ -1,67 +1,96 @@
 <?xml version="1.0"?>
-<robot xmlns:xacro="http://www.ros.org/wiki/xacro" name="robot_2030a">
+<robot xmlns:xacro="http://www.ros.org/wiki/xacro" name="mycobot_320pi">
     <ros2_control name="RobotSystem" type="system">
         <xacro:property name="PI" value="3.14159265359" />
         <!-- ros2_control Gazebo -->
         <xacro:if value="$(arg is_sim)">
-            <hardware>
-                <plugin>gazebo_ros2_control/GazeboSystem</plugin>
-            </hardware>
+            <!-- ROS 2 Humble -->
+            <xacro:if value="$(arg is_ignition)">
+                <hardware>
+                    <plugin>ign_ros2_control/IgnitionSystem</plugin>
+                </hardware>
+            </xacro:if>
+            <!-- ROS 2 Iron or above -->
+            <xacro:unless value="$(arg is_ignition)">
+                <hardware>
+                    <plugin>gz_ros2_control/GazeboSimSystem</plugin>
+                </hardware>
+            </xacro:unless>
+            <joint name="left_jaw_joint_2">
+                <param name="mimic">left_jaw_joint_1</param>
+                <param name="multiplier">1</param>
+            </joint>
+            <joint name="left_jaw_joint_3">
+                <param name="mimic">left_jaw_joint_1</param>
+                <param name="multiplier">-1</param>
+            </joint>
+            <joint name="right_jaw_joint_1">
+                <param name="mimic">left_jaw_joint_1</param>
+                <param name="multiplier">-1</param>
+            </joint>
+            <joint name="right_jaw_joint_2">
+                <param name="mimic">left_jaw_joint_1</param>
+                <param name="multiplier">-1</param>
+            </joint>
+            <joint name="right_jaw_joint_3">
+                <param name="mimic">left_jaw_joint_1</param>
+                <param name="multiplier">1</param>
+            </joint>
         </xacro:if>
         <!-- ros2_control Real Robot -->
         <xacro:unless value="$(arg is_sim)">
             <hardware>
-                <plugin>mycobot_320pi_controller/Mycobot_320pi_Interface</plugin>
+                <plugin>mycobot_320pi_controller/Mycobot320piInterface</plugin>
                 <param name="port">/dev/ttyACM0</param>
             </hardware>
         </xacro:unless>
+        <!-- Joint 1 -->
         <joint name="joint_1">
-            <command_interface name="position">
-            <param name="min">-${PI / 2}</param>
-            <param name="max">${PI / 2}</param>
-            </command_interface>
+            <command_interface name="position"/>
             <state_interface name="position"/>
+            <param name="min_position">-2.93</param>
+            <param name="max_position">2.93</param>
         </joint>
+        <!-- Joint 2 -->
         <joint name="joint_2">
-            <command_interface name="position">
-            <param name="min">-${PI / 2}</param>
-            <param name="max">${PI / 2}</param>
-            </command_interface>
+            <command_interface name="position"/>
             <state_interface name="position"/>
+            <param name="min_position">-2.35</param>
+            <param name="max_position">2.35</param>
         </joint>
+        <!-- Joint 3 -->
         <joint name="joint_3">
-            <command_interface name="position">
-            <param name="min">-${PI / 2}</param>
-            <param name="max">${PI / 2}</param>
-            </command_interface>
+            <command_interface name="position"/>
             <state_interface name="position"/>
+            <param name="min_position">-2.53</param>
+            <param name="max_position">2.53</param>
         </joint>
+        <!-- Joint 4 -->
         <joint name="joint_4">
-            <command_interface name="position">
-            <param name="min">-${PI / 2}</param>
-            <param name="max">0.0</param>
-            </command_interface>
+            <command_interface name="position"/>
             <state_interface name="position"/>
+            <param name="min_position">-2.53</param>
+            <param name="max_position">2.53</param>
         </joint>
+        <!-- Joint 5 -->
         <joint name="joint_5">
-            <command_interface name="position">
-            <param name="min">-${PI / 2}</param>
-            <param name="max">0.0</param>
-            </command_interface>
+            <command_interface name="position"/>
             <state_interface name="position"/>
+            <param name="min_position">-2.93</param>
+            <param name="max_position">2.93</param>
         </joint>
+        <!-- Joint 6 -->
         <joint name="joint_6">
-            <command_interface name="position">
-            <param name="min">-${PI / 2}</param>
-            <param name="max">0.0</param>
-            </command_interface>
+            <command_interface name="position"/>
             <state_interface name="position"/>
+            <param name="min_position">-3.14</param>
+            <param name="max_position">3.14</param>
         </joint>
+        <!-- Gripper Master Joint -->
         <joint name="left_jaw_joint_1">
-            <command_interface name="position">
-                <param name="min">-1.11</param>
-                <param name="max">0.0</param>
-            </command_interface>
+            <command_interface name="position"/>
             <state_interface name="position"/>
+            <param name="min_position">-1.11</param>
+            <param name="max_position">0.0</param>
         </joint>
     </ros2_control>

Commit message: push

File: brain_pc/src/mycobot_320pi_description/urdf/mycobot_320pi.urdf.xacro (robot description, xacro)
@@ -125,5 +125,5 @@
         <xacro:default_inertial mass="1.0"/>
         <visual>
-            <origin xyz="0 0 0" rpy="0 0 0"/>
+            <origin xyz="0 0 0" rpy="0 -0.9599 0"/>
             <geometry>
                 <mesh filename="package://mycobot_320pi_description/meshes/link_6.dae"/>
@@ -131,5 +131,5 @@
         </visual>
         <collision>
-            <origin xyz="0 0 0" rpy="0 0 0"/>
+            <origin xyz="0 0 0" rpy="0 -0.9599 0"/>
             <geometry>
                 <mesh filename="package://mycobot_320pi_description/meshes/link_6.dae"/>
@@ -300,5 +300,5 @@
         <child link = "link_2"/>
         <origin xyz="0 -0.0477 0.079" rpy="0 0 0"/>
-        <axis xyz="0 1 0"/>
+        <axis xyz="0 -1 0"/>
         <limit lower="-2.35" upper="2.35" effort="5" velocity="10.0"/>
     </joint>
@@ -308,5 +308,5 @@
         <child link = "link_3"/>
         <origin xyz="0.0 0.0075 0.135" rpy="0 0 0"/>
-        <axis xyz="0 1 0"/>
+        <axis xyz="0 -1 0"/>
         <limit lower="-2.53" upper="2.53" effort="5" velocity="10.0"/>
     </joint>
@@ -316,5 +316,5 @@
         <child link = "link_4"/>
         <origin xyz="0.0 0.002 0.1201" rpy="0 0 0"/>
-        <axis xyz="0 1 0"/>
+        <axis xyz="0 -1 0"/>
         <limit lower="-2.53" upper="2.53" effort="5" velocity="10.0"/>
     </joint>
@@ -331,6 +331,6 @@
         <parent link="link_5"/>
         <child link = "link_6"/>
-        <origin xyz="0.0 -0.045 0.05" rpy="0 0 0"/>
-        <axis xyz="0 1 0"/>
+        <origin xyz="0.0 -0.045 0.05" rpy="0 -2.3662 0"/>
+        <axis xyz="0 -1 0"/>
         <limit lower="-3.14" upper="3.14" effort="5" velocity="10.0"/>
     </joint>
